File: hardware/instrumentation.sch (KiCad schematic (older format))
At the start: 0 parts

Commit message: Added Instrumentation Components To Kicad
Added SN74HCS153, LMV554, and TMP235.
Parts:
- added U?: LMV554, symbol mallard:LMV554
- added U?: SN74HCS153, symbol mallard:SN74HCS153
- added U? (x3): TMP235, symbol mallard:TMP235
Changed lines of the file:
@@
 $Descr A4 11693 8268
 encoding utf-8
-Sheet 1 3
+Sheet 3 4
 Title ""
 Date ""
@@
 Comment4 ""
 $EndDescr
+$Comp
+L mallard:LMV554 U?
+U 1 1 60F26055
+P 3150 2700
+F 0 "U?" H 3150 2925 50  0000 C CNN
+F 1 "LMV554" H 3150 2834 50  0000 C CNN
+F 2 "" H 3150 1850 50  0001 C CNN
+F 3 "https://www.ti.com/lit/ds/symlink/lmv551.pdf?HQS=dis-dk-null-digikeymode-dsf-pf-null-wwe&ts=1626469395066&ref_url=https%253A%252F%252Fwww.ti.com%252Fgeneral%252Fdocs%252Fsuppproductinfo.tsp%253FdistId%253D10%2526gotoUrl%253Dhttps%253A%252F%252Fwww.ti.com%252Flit%252Fgpn%252Flmv551" H 3150 1850 50  0001 C CNN
+	1    3150 2700
+	1    0    0    -1
+$EndComp
+$Comp
+L mallard:SN74HCS153 U?
+U 1 1 60F271CF
+P 4650 2700
+F 0 "U?" H 4650 2925 50  0000 C CNN
+F 1 "SN74HCS153" H 4650 2834 50  0000 C CNN
+F 2 "" H 4650 2800 50  0001 C CNN
+F 3 "" H 4650 2800 50  0001 C CNN
+	1    4650 2700
+	1    0    0    -1
+$EndComp
+$Comp
+L mallard:TMP235 U?
+U 1 1 60F2A653
+P 6250 2700
+F 0 "U?" H 6250 2875 50  0000 C CNN
+F 1 "TMP235" H 6250 2784 50  0000 C CNN
+F 2 "" H 6250 2250 50  0001 C CNN
+F 3 "" H 6250 2250 50  0001 C CNN
+	1    6250 2700
+	1    0    0    -1
+$EndComp
+$Comp
+L mallard:TMP235 U?
+U 1 1 60F2B7FB
+P 6250 3450
+F 0 "U?" H 6250 3625 50  0000 C CNN
+F 1 "TMP235" H 6250 3534 50  0000 C CNN
+F 2 "" H 6250 3000 50  0001 C CNN
+F 3 "" H 6250 3000 50  0001 C CNN
+	1    6250 3450
+	1    0    0    -1
+$EndComp
+$Comp
+L mallard:TMP235 U?
+U 1 1 60F2C19D
+P 6250 4200
+F 0 "U?" H 6250 4375 50  0000 C CNN
+F 1 "TMP235" H 6250 4284 50  0000 C CNN
+F 2 "" H 6250 3750 50  0001 C CNN
+F 3 "" H 6250 3750 50  0001 C CNN
+	1    6250 4200
+	1    0    0    -1
+$EndComp
 $EndSCHEMATC
