File: hardware/instrumentation.sch (KiCad schematic (older format))
At the start: 19 parts, among them U500 LMV554, U600 TMUX1309, U700 TMUX1309

Commit message: Finished adding TMP sensors and footprints
Parts:
- removed Ref1: Ref Electrode, symbol Connector_Generic:Conn_01x01
- added C10, C8, C9: 1uF, Capacitor_SMD:C_0603_1608Metric_Pad1.08x0.95mm_HandSolder, symbol mallard-rescue:C-Device
- added R100, R101: Jumper, Resistor_SMD:R_0603_1608Metric_Pad0.98x0.95mm_HandSolder, symbol mallard-rescue:R_Small-Device
- added Ref1: Conn_01x02, Connector_Coaxial:BNC_TEConnectivity_1478204_Vertical, symbol Connector_Generic:Conn_01x02
- added U2, U3, U4: TMP235, Connector_PinHeader_2.54mm:PinHeader_1x05_P2.54mm_Vertical, symbol mallard:TMP235
- Eh1: renamed from Eh603; footprint (none) -> Connector_PinHeader_2.54mm:PinHeader_1x01_P2.54mm_Vertical; symbol Connector_Generic:Conn_01x01 -> mallard-rescue:Conn_01x01-Connector_Generic
- Eh2: renamed from Eh604; footprint (none) -> Connector_PinHeader_2.54mm:PinHeader_1x01_P2.54mm_Vertical; symbol Connector_Generic:Conn_01x01 -> mallard-rescue:Conn_01x01-Connector_Generic
- Eh3: renamed from Eh605; footprint (none) -> Connector_PinHeader_2.54mm:PinHeader_1x01_P2.54mm_Vertical; symbol Connector_Generic:Conn_01x01 -> mallard-rescue:Conn_01x01-Connector_Generic
- R10: renamed from R504; symbol Device:R -> mallard-rescue:R-Device
- R11: renamed from R506; symbol Device:R -> mallard-rescue:R-Device
- R3: renamed from R600; symbol Device:R -> mallard-rescue:R-Device
- R4: renamed from R500; symbol Device:R -> mallard-rescue:R-Device
- R5: renamed from R507; symbol Device:R -> mallard-rescue:R-Device
- R6: renamed from R505; symbol Device:R -> mallard-rescue:R-Device
- R7: renamed from R501; symbol Device:R -> mallard-rescue:R-Device
- R8: renamed from R502; symbol Device:R -> mallard-rescue:R-Device
- R9: renamed from R503; symbol Device:R -> mallard-rescue:R-Device
- SM1: renamed from SM600; symbol Connector_Generic:Conn_01x03 -> mallard-rescue:Conn_01x03-Connector_Generic
- SM2: renamed from SM601; symbol Connector_Generic:Conn_01x03 -> mallard-rescue:Conn_01x03-Connector_Generic
- SM3: renamed from SM602; symbol Connector_Generic:Conn_01x03 -> mallard-rescue:Conn_01x03-Connector_Generic
- renumbered U600 to U5, U700 to U6, U500 to U7
Connections:
- net +3V3: now also C10.1, C8.1, C9.1, U2.4 (VCC), U3.4 (VCC), U4.4 (VCC)
- net GND: now also C10.2, C8.2, C9.2, U2.2 (GND), U3.2 (GND), U4.2 (GND)
- net at U7.12 (IN_D+): now also R100.1, R101.1
- net at U6.12 (S0A): now also U2.3 (Vout)
- net at U6.14 (S1A): now also U3.3 (Vout)
- net at U6.15 (S2A): now also U4.3 (Vout)
- new net: R100.2, Ref1.1 (Pin_1)
- new net: R101.2, Ref1.2 (Pin_2)
Other:
- note added: "FOOTPRINT FOR TMP235 IS 5 HOLE CONNECTOR"
- note removed: "Needed New Temp sensors\n"
