File: hardware/power.sch (KiCad schematic (older format))
At the start: 23 parts, among them U100 BQ24210DQCT, U200 LTC1983ES6-3, U300 TPS717

Commit message: Added more ref des
Parts:
- renumbered R10x to R10x1
Changed lines of the file:
@@
 	8900 3200 8800 3200
 $Comp
-L power:-3V3 #PWR?
+L power:-3V3 #PWR0107
 U 1 1 6161FA5E
 P 11000 3000
-F 0 "#PWR?" H 11000 3100 50  0001 C CNN
+F 0 "#PWR0107" H 11000 3100 50  0001 C CNN
 F 1 "-3V3" V 11015 3128 50  0000 L CNN
 F 2 "" H 11000 3000 50  0001 C CNN
@@
 $EndComp
 $Comp
-L power:GND #PWR?
+L power:GND #PWR0108
 U 1 1 615BBB45
 P 9600 5250
-F 0 "#PWR?" H 9600 5000 50  0001 C CNN
+F 0 "#PWR0108" H 9600 5000 50  0001 C CNN
 F 1 "GND" V 9605 5122 50  0000 R CNN
 F 2 "" H 9600 5250 50  0001 C CNN
@@
 $EndComp
 $Comp
-L power:GND #PWR?
+L power:GND #PWR0109
 U 1 1 615C9273
 P 10100 5250
-F 0 "#PWR?" H 10100 5000 50  0001 C CNN
+F 0 "#PWR0109" H 10100 5000 50  0001 C CNN
 F 1 "GND" H 10105 5077 50  0000 C CNN
 F 2 "" H 10100 5250 50  0001 C CNN
@@
 $EndComp
 $Comp
-L power:+1V0 #PWR?
+L power:+1V0 #PWR0110
 U 1 1 615CDF04
 P 10800 4400
-F 0 "#PWR?" H 10800 4250 50  0001 C CNN
+F 0 "#PWR0110" H 10800 4250 50  0001 C CNN
 F 1 "+1V0" H 10815 4573 50  0000 C CNN
 F 2 "" H 10800 4400 50  0001 C CNN
@@
 $EndComp
 $Comp
-L power:+3V3 #PWR?
+L power:+3V3 #PWR0111
 U 1 1 615DFBEC
 P 7750 4400
-F 0 "#PWR?" H 7750 4250 50  0001 C CNN
+F 0 "#PWR0111" H 7750 4250 50  0001 C CNN
 F 1 "+3V3" H 7765 4573 50  0000 C CNN
 F 2 "" H 7750 4400 50  0001 C CNN
@@
 	7900 4800 7900 4850
 $Comp
-L power:GND #PWR?
+L power:GND #PWR0112
 U 1 1 6193F3E7
 P 7900 4850
-F 0 "#PWR?" H 7900 4600 50  0001 C CNN
+F 0 "#PWR0112" H 7900 4600 50  0001 C CNN
 F 1 "GND" V 7905 4722 50  0000 R CNN
 F 2 "" H 7900 4850 50  0001 C CNN
@@
 	7300 3000 7300 2950
 $Comp
-L power:+3V3 #PWR?
+L power:+3V3 #PWR0113
 U 1 1 61970B46
 P 7750 2950
-F 0 "#PWR?" H 7750 2800 50  0001 C CNN
+F 0 "#PWR0113" H 7750 2800 50  0001 C CNN
 F 1 "+3V3" H 7765 3123 50  0000 C CNN
 F 2 "" H 7750 2950 50  0001 C CNN
@@
 	9600 3000 10350 3000
 $Comp
-L power:GND #PWR?
+L power:GND #PWR0114
 U 1 1 619CB529
 P 10350 3600
-F 0 "#PWR?" H 10350 3350 50  0001 C CNN
+F 0 "#PWR0114" H 10350 3350 50  0001 C CNN
 F 1 "GND" H 10355 3427 50  0000 C CNN
 F 2 "" H 10350 3600 50  0001 C CNN
@@
 $EndComp
 $Comp
-L Device:R R10x
+L Device:R R10x1
 U 1 1 619D521F
 P 2900 4250
-F 0 "R10x" H 2970 4296 50  0000 L CNN
+F 0 "R10x1" H 2970 4296 50  0000 L CNN
 F 1 "5.1k" H 2970 4205 50  0000 L CNN
 F 2 "Resistor_SMD:R_0603_1608Metric_Pad0.98x0.95mm_HandSolder" V 2830 4250 50  0001 C CNN
@@
 Connection ~ 4250 3900
 $Comp
-L power:GND #PWR?
+L power:GND #PWR0115
 U 1 1 619EC3D6
 P 4250 4600
-F 0 "#PWR?" H 4250 4350 50  0001 C CNN
+F 0 "#PWR0115" H 4250 4350 50  0001 C CNN
 F 1 "GND" H 4255 4427 50  0000 C CNN
 F 2 "" H 4250 4600 50  0001 C CNN

Commit message: Finished adding TMP sensors and footprints
Parts:
- BatteryPack1: symbol Device:Battery_Cell -> mallard-rescue:Battery_Cell-Device
- C11: renamed from C100; symbol Device:C -> mallard-rescue:C-Device
- C12: renamed from C101; symbol Device:C -> mallard-rescue:C-Device
- C13: renamed from C200; symbol Device:C -> mallard-rescue:C-Device
- C14: renamed from C300; symbol Device:C -> mallard-rescue:C-Device
- C15: renamed from C201; footprint (none) -> Capacitor_SMD:C_0603_1608Metric_Pad1.08x0.95mm_HandSolder; symbol Device:C -> mallard-rescue:C-Device; Digikey 311-1446-1-ND -> 1276-1019-1-ND
- C16: renamed from C301; symbol Device:C -> mallard-rescue:C-Device
- C17: renamed from C202; symbol Device:C -> mallard-rescue:C-Device
- D2: renamed from D100; symbol Device:D -> mallard-rescue:D-Device
- D3: renamed from D101; symbol Device:LED -> mallard-rescue:LED-Device
- D4: renamed from D102; symbol Device:LED -> mallard-rescue:LED-Device
- R10x1: symbol Device:R -> mallard-rescue:R-Device
- R12: renamed from R100; symbol Device:R -> mallard-rescue:R-Device
- R13: renamed from R103; symbol Device:R -> mallard-rescue:R-Device
- R14: renamed from R101; symbol Device:R -> mallard-rescue:R-Device
- R15: renamed from R102; symbol Device:R -> mallard-rescue:R-Device
- R16: renamed from R300; symbol Device:R -> mallard-rescue:R-Device
- R17: renamed from R301; symbol Device:R -> mallard-rescue:R-Device
- R18: renamed from R303; symbol Device:R_Small -> mallard-rescue:R_Small-Device
- TH1: renamed from TH100; footprint (none) -> Resistor_THT:R_Axial_DIN0204_L3.6mm_D1.6mm_P2.54mm_Vertical; symbol Device:Thermistor -> mallard-rescue:Thermistor-Device
- U9: renamed from U300; value TPS717 -> TPS71710DRVR; footprint (none) -> Package_SON:WSON-6-1EP_2x2mm_P0.65mm_EP1x1.6mm; Digikey 296-27043-1-ND -> 296-22984-1-ND
- renumbered U200 to U10, U100 to U8
Connections:
- wire segments 69 -> 72
Other:
- note added: "May have to find alt thermistor...\nNeed B=3435K"
