File: hardware/microcontroiller.sch (KiCad schematic (older format))
At the start: 0 parts

Commit message: Added all Digikey part numbers. Started MC schematic. Fixed the reference number on some symbols.
Parts:
- added C1, C2: 20pF, symbol Device:C_Small
- added C3, C4, C5, C6: 0.1uF, symbol Device:C_Small
- added D1: Orange, symbol Device:LED_Small
- added J1: SWD, symbol Connector_Generic:Conn_02x05_Odd_Even
- added J2: USB_A, symbol Connector:USB_A
- added R1: 10k, symbol Device:R_Small
- added R2: 680, symbol Device:R_Small
- added SW1: RESET Switch, symbol Switch:SW_Push_Open_Dual
- added U1: STM32L431CBTx, Package_QFP:LQFP-48_7x7mm_P0.5mm, symbol MCU_ST_STM32L4:STM32L431CBTx
- added Y1: 32.768kHz, symbol Device:Crystal_Small
Connections:
- net labels added: +3V3, +5V, 3V3_VDD, GND, RESET_L, SWCLK, SWDIO, USB+, USB-
- wire segments 0 -> 63
- no-connect marks 0 -> 3
Other:
- note added: "Check Symbol with Datasheet to make sure pins match"
