File: hardware/mallard.sch (KiCad schematic (older format))
At the start: 84 parts, among them J1 USB_A, J2 Conn_02x03_Odd_Even, J3 Conn_01x03, SW1 RESET Switch, U1 TMP235, U10 LTC1983ES6-3, U11 STM32L4Q5xx, U2 TMP235, U3 TMP235, U4 BQ24210DQCT, U5 TMUX1309, U6 TMUX1309, U7 LMP7721, U8 TPS71710DRVR, U9 LMV554

Commit message: Schematic and Layout Finished
Needs review
Parts:
- L1: renamed from L?; Digikey ASMCI-0805-4R7M-T -> 490-7782-1-ND
- gave numbers to parts that had none: 10
Changed lines of the file:
@@
 	-700 9150 800  9150
 $Comp
-L Connector_Generic:Conn_01x03 J?
+L Connector_Generic:Conn_01x03 J4
 U 1 1 61FF33B4
 P -3950 12500
-F 0 "J?" H -4032 12175 50  0000 C CNN
+F 0 "J4" H -4032 12175 50  0000 C CNN
 F 1 "Conn_01x03" H -4032 12266 50  0000 C CNN
 F 2 "Connector_PinHeader_2.54mm:PinHeader_1x03_P2.54mm_Vertical" H -3950 12500 50  0001 C CNN
@@
 	-3750 12500 -2600 12500
 $Comp
-L Connector_Generic:Conn_01x03 J?
+L Connector_Generic:Conn_01x03 J5
 U 1 1 620584BA
 P -3700 13500
-F 0 "J?" H -3782 13175 50  0000 C CNN
+F 0 "J5" H -3782 13175 50  0000 C CNN
 F 1 "Conn_01x03" H -3782 13266 50  0000 C CNN
 F 2 "Connector_PinHeader_2.54mm:PinHeader_1x03_P2.54mm_Vertical" H -3700 13500 50  0001 C CNN
@@
 AR Path="/60B3FF2D/6205C36F" Ref="#PWR?"  Part="1"
 AR Path="/60B3FE92/6205C36F" Ref="#PWR?"  Part="1"
-AR Path="/6205C36F" Ref="#PWR?"  Part="1"
-F 0 "#PWR?" H -3500 14150 50  0001 C CNN
+AR Path="/6205C36F" Ref="#PWR0133"  Part="1"
+F 0 "#PWR0133" H -3500 14150 50  0001 C CNN
 F 1 "GND" H -3495 14227 50  0000 C CNN
 F 2 "" H -3500 14400 50  0001 C CNN
@@
 AR Path="/60B3FF2D/6205C376" Ref="C?"  Part="1"
 AR Path="/60B3FE92/6205C376" Ref="C?"  Part="1"
-AR Path="/6205C376" Ref="C?"  Part="1"
-F 0 "C?" H -3285 14796 50  0000 L CNN
+AR Path="/6205C376" Ref="C3"  Part="1"
+F 0 "C3" H -3285 14796 50  0000 L CNN
 F 1 "1uF" H -3285 14705 50  0000 L CNN
 F 2 "Capacitor_SMD:C_0603_1608Metric_Pad1.08x0.95mm_HandSolder" H -3362 14600 50  0001 C CNN
@@
 P -3400 14900
 AR Path="/60B3FE92/6205C37C" Ref="#PWR?"  Part="1"
-AR Path="/6205C37C" Ref="#PWR?"  Part="1"
-F 0 "#PWR?" H -3400 14650 50  0001 C CNN
+AR Path="/6205C37C" Ref="#PWR0135"  Part="1"
+F 0 "#PWR0135" H -3400 14650 50  0001 C CNN
 F 1 "GND" H -3395 14727 50  0000 C CNN
 F 2 "" H -3400 14900 50  0001 C CNN
@@
 P -3300 14600
 AR Path="/60B3FE92/6205C382" Ref="#PWR?"  Part="1"
-AR Path="/6205C382" Ref="#PWR?"  Part="1"
-F 0 "#PWR?" H -3300 14450 50  0001 C CNN
+AR Path="/6205C382" Ref="#PWR0136"  Part="1"
+F 0 "#PWR0136" H -3300 14450 50  0001 C CNN
 F 1 "+3V3" H -3285 14773 50  0000 C CNN
 F 2 "" H -3300 14600 50  0001 C CNN
@@
 $EndComp
 $Comp
-L Connector_Generic:Conn_01x03 J?
+L Connector_Generic:Conn_01x03 J6
 U 1 1 6205C388
 P -3700 14500
-F 0 "J?" H -3782 14175 50  0000 C CNN
+F 0 "J6" H -3782 14175 50  0000 C CNN
 F 1 "Conn_01x03" H -3782 14266 50  0000 C CNN
 F 2 "Connector_PinHeader_2.54mm:PinHeader_1x03_P2.54mm_Vertical" H -3700 14500 50  0001 C CNN
@@
 AR Path="/60B3FF2D/620BF937" Ref="C?"  Part="1"
 AR Path="/60B3FE92/620BF937" Ref="C?"  Part="1"
-AR Path="/620BF937" Ref="C?"  Part="1"
-F 0 "C?" H -3285 13796 50  0000 L CNN
+AR Path="/620BF937" Ref="C2"  Part="1"
+F 0 "C2" H -3285 13796 50  0000 L CNN
 F 1 "1uF" H -3285 13705 50  0000 L CNN
 F 2 "Capacitor_SMD:C_0603_1608Metric_Pad1.08x0.95mm_HandSolder" H -3362 13600 50  0001 C CNN
@@
 P -3400 13900
 AR Path="/60B3FE92/620BF93D" Ref="#PWR?"  Part="1"
-AR Path="/620BF93D" Ref="#PWR?"  Part="1"
-F 0 "#PWR?" H -3400 13650 50  0001 C CNN
+AR Path="/620BF93D" Ref="#PWR0138"  Part="1"
+F 0 "#PWR0138" H -3400 13650 50  0001 C CNN
 F 1 "GND" H -3395 13727 50  0000 C CNN
 F 2 "" H -3400 13900 50  0001 C CNN
@@
 P -3300 13600
 AR Path="/60B3FE92/620BF943" Ref="#PWR?"  Part="1"
-AR Path="/620BF943" Ref="#PWR?"  Part="1"
-F 0 "#PWR?" H -3300 13450 50  0001 C CNN
+AR Path="/620BF943" Ref="#PWR0139"  Part="1"
+F 0 "#PWR0139" H -3300 13450 50  0001 C CNN
 F 1 "+3V3" H -3285 13773 50  0000 C CNN
 F 2 "" H -3300 13600 50  0001 C CNN
@@
 Wrong footprint size
 $Comp
-L mallard:LTC3529EDCB U?
+L mallard:LTC3529EDCB U12
 U 1 1 62066D6A
 P 2400 5950
-F 0 "U?" H 2750 6125 50  0000 C CNN
+F 0 "U12" H 2750 6125 50  0000 C CNN
 F 1 "LTC3529EDCB" H 2750 6034 50  0000 C CNN
 F 2 "mallard:DFN200X300X80-9N" H 2300 6100 50  0001 C CNN
@@
 $EndComp
 $Comp
-L Device:C_Small C?
+L Device:C_Small C22
 U 1 1 62068D50
 P 1750 5850
-F 0 "C?" H 1550 5900 50  0000 L CNN
+F 0 "C22" H 1550 5900 50  0000 L CNN
 F 1 "3.3uF" H 1450 5800 50  0000 L CNN
 F 2 "Capacitor_SMD:C_0603_1608Metric_Pad1.08x0.95mm_HandSolder" H 1750 5850 50  0001 C CNN
@@
 $EndComp
 $Comp
-L power:+3V3 #PWR?
+L power:+3V3 #PWR0169
 U 1 1 6209B3D5
 P 1750 5700
-F 0 "#PWR?" H 1750 5550 50  0001 C CNN
+F 0 "#PWR0169" H 1750 5550 50  0001 C CNN
 F 1 "+3V3" H 1765 5873 50  0000 C CNN
 F 2 "" H 1750 5700 50  0001 C CNN
@@
 $EndComp
 $Comp
-L power:+5V #PWR?
+L power:+5V #PWR0170
 U 1 1 6209C408
 P 3600 6300
-F 0 "#PWR?" H 3600 6150 50  0001 C CNN
+F 0 "#PWR0170" H 3600 6150 50  0001 C CNN
 F 1 "+5V" H 3615 6473 50  0000 C CNN
 F 2 "" H 3600 6300 50  0001 C CNN
@@
 $EndComp
 $Comp
-L power:GND #PWR?
+L power:GND #PWR0171
 U 1 1 6209E0C4
 P 1750 5950
-F 0 "#PWR?" H 1750 5700 50  0001 C CNN
+F 0 "#PWR0171" H 1750 5700 50  0001 C CNN
 F 1 "GND" H 1755 5777 50  0000 C CNN
 F 2 "" H 1750 5950 50  0001 C CNN
@@
 $EndComp
 $Comp
-L Device:R_Small R?
+L Device:R_Small R25
 U 1 1 620BA7E6
 P 2150 6200
-F 0 "R?" V 1950 6200 50  0000 C CNN
+F 0 "R25" V 1950 6200 50  0000 C CNN
 F 1 "370" V 2050 6200 50  0000 C CNN
 F 2 "Resistor_SMD:R_0603_1608Metric_Pad0.98x0.95mm_HandSolder" H 2150 6200 50  0001 C CNN
@@
 Connection ~ 1750 5750
 $Comp
-L Device:C_Small C?
+L Device:C_Small C23
 U 1 1 6213E3BD
 P 3600 6400
-F 0 "C?" H 3692 6446 50  0000 L CNN
+F 0 "C23" H 3692 6446 50  0000 L CNN
 F 1 "10uF" H 3692 6355 50  0000 L CNN
 F 2 "Capacitor_SMD:C_0603_1608Metric_Pad1.08x0.95mm_HandSolder" H 3600 6400 50  0001 C CNN
@@
 $EndComp
 $Comp
-L power:GND #PWR?
+L power:GND #PWR0172
 U 1 1 62158AAE
 P 3600 6500
-F 0 "#PWR?" H 3600 6250 50  0001 C CNN
+F 0 "#PWR0172" H 3600 6250 50  0001 C CNN
 F 1 "GND" H 3605 6327 50  0000 C CNN
 F 2 "" H 3600 6500 50  0001 C CNN
@@
 Connection ~ 3600 6300
 $Comp
-L power:GND #PWR?
+L power:GND #PWR0173
 U 1 1 62173E2F
 P 3200 6150
-F 0 "#PWR?" H 3200 5900 50  0001 C CNN
+F 0 "#PWR0173" H 3200 5900 50  0001 C CNN
 F 1 "GND" V 3205 6022 50  0000 R CNN
 F 2 "" H 3200 6150 50  0001 C CNN
@@
 $EndComp
 $Comp
-L Device:L L?
+L Device:L L1
 U 1 1 6218F7E1
 P 2750 5650
-F 0 "L?" V 2940 5650 50  0000 C CNN
+F 0 "L1" V 2940 5650 50  0000 C CNN
 F 1 "4.7uH" V 2849 5650 50  0000 C CNN
 F 2 "Inductor_SMD:L_0805_2012Metric_Pad1.05x1.20mm_HandSolder" H 2750 5650 50  0001 C CNN
 F 3 "~" H 2750 5650 50  0001 C CNN
-F 4 "ASMCI-0805-4R7M-T" V 2750 5650 50  0001 C CNN "Digikey"
+F 4 "490-7782-1-ND" V 2750 5650 50  0001 C CNN "Digikey"
 	1    2750 5650
 	0    -1   -1   0
@@
 	3200 6500 3600 6500
 $Comp
-L Device:D_Small D?
+L Device:D_Small D5
 U 1 1 6209F53B
 P 1950 5850
-F 0 "D?" V 1996 5782 50  0000 R CNN
+F 0 "D5" V 1996 5782 50  0000 R CNN
 F 1 "RED" V 1905 5782 50  0000 R CNN
 F 2 "LED_SMD:LED_0603_1608Metric_Pad1.05x0.95mm_HandSolder" V 1950 5850 50  0001 C CNN

Commit message: Updated footprints
Parts:
- D4: footprint Resistor_SMD:R_0805_2012Metric_Pad1.20x1.40mm_HandSolder -> Diode_SMD:D_0805_2012Metric_Castellated
- R10, R13, R14, R15, R16, R17, R18, R19, R24, R4, R6, R8: footprint Resistor_SMD:R_0201_0603Metric_Pad0.64x0.40mm_HandSolder -> Resistor_SMD:R_0603_1608Metric_Pad0.98x0.95mm_HandSolder
Changed lines of the file:
@@
 F 0 "R24" V 17254 2300 50  0000 C CNN
 F 1 "10k" V 17345 2300 50  0000 C CNN
-F 2 "Resistor_SMD:R_0201_0603Metric_Pad0.64x0.40mm_HandSolder" H 17450 2300 50  0001 C CNN
+F 2 "Resistor_SMD:R_0603_1608Metric_Pad0.98x0.95mm_HandSolder" H 17450 2300 50  0001 C CNN
 F 3 "https://www.yageo.com/upload/media/product/productsearch/datasheet/rchip/PYu-RC_Group_51_RoHS_L_11.pdf" H 17450 2300 50  0001 C CNN
 F 4 "13-RC0603DR-0710KLCT-ND‎" V 17450 2300 50  0001 C CNN "Digikey"
@@
 F 0 "D4" H 15900 6050 50  0000 C CNN
 F 1 "Orange" H 15900 6150 50  0000 C CNN
-F 2 "Resistor_SMD:R_0805_2012Metric_Pad1.20x1.40mm_HandSolder" V 15900 6250 50  0001 C CNN
+F 2 "Diode_SMD:D_0805_2012Metric_Castellated" V 15900 6250 50  0001 C CNN
 F 3 "https://optoelectronics.liteon.com/upload/download/DS-22-99-0185/LTST-C170KFKT.pdf" V 15900 6250 50  0001 C CNN
 F 4 "160-1413-1-ND" H 15900 6250 50  0001 C CNN "Digikey"
@@
 F 0 "R4" V -857 10550 50  0000 C CNN
 F 1 "10k" V -766 10550 50  0000 C CNN
-F 2 "Resistor_SMD:R_0201_0603Metric_Pad0.64x0.40mm_HandSolder" V -720 10550 50  0001 C CNN
+F 2 "Resistor_SMD:R_0603_1608Metric_Pad0.98x0.95mm_HandSolder" V -720 10550 50  0001 C CNN
 F 3 "https://www.yageo.com/upload/media/product/productsearch/datasheet/rchip/PYu-RC_Group_51_RoHS_L_11.pdf" H -650 10550 50  0001 C CNN
 F 4 "13-RC0603DR-0710KLCT-ND‎" V -650 10550 50  0001 C CNN "Digikey"
@@
 F 0 "R16" V 3243 9450 50  0000 C CNN
 F 1 "20k DNI" V 3334 9450 50  0000 C CNN
-F 2 "Resistor_SMD:R_0201_0603Metric_Pad0.64x0.40mm_HandSolder" V 3380 9450 50  0001 C CNN
+F 2 "Resistor_SMD:R_0603_1608Metric_Pad0.98x0.95mm_HandSolder" V 3380 9450 50  0001 C CNN
 F 3 "https://industrial.panasonic.com/cdbs/www-data/pdf/RDM0000/AOA0000C328.pdf" H 3450 9450 50  0001 C CNN
 F 4 "‎P20429CT-ND‎" V 3450 9450 50  0001 C CNN "Digikey"
@@
 F 0 "R15" V 3243 9050 50  0000 C CNN
 F 1 "30k" V 3334 9050 50  0000 C CNN
-F 2 "Resistor_SMD:R_0201_0603Metric_Pad0.64x0.40mm_HandSolder" V 3380 9050 50  0001 C CNN
+F 2 "Resistor_SMD:R_0603_1608Metric_Pad0.98x0.95mm_HandSolder" V 3380 9050 50  0001 C CNN
 F 3 "https://www.yageo.com/upload/media/product/productsearch/datasheet/rchip/PYu-RT_1-to-0.01_RoHS_L_12.pdf" H 3450 9050 50  0001 C CNN
 F 4 "311-30KDCT-ND‎" V 3450 9050 50  0001 C CNN "Digikey"
@@
 F 0 "R14" H 3120 12846 50  0000 L CNN
 F 1 "1k" H 3120 12755 50  0000 L CNN
-F 2 "Resistor_SMD:R_0201_0603Metric_Pad0.64x0.40mm_HandSolder" V 2980 12800 50  0001 C CNN
+F 2 "Resistor_SMD:R_0603_1608Metric_Pad0.98x0.95mm_HandSolder" V 2980 12800 50  0001 C CNN
 F 3 "https://www.vishay.com/docs/20065/rcse3.pdf" H 3050 12800 50  0001 C CNN
 F 4 "541-2788-1-ND" H 3050 12800 50  0001 C CNN "Digikey"
@@
 F 0 "R18" V 3293 12550 50  0000 C CNN
 F 1 "9.1k" V 3384 12550 50  0000 C CNN
-F 2 "Resistor_SMD:R_0201_0603Metric_Pad0.64x0.40mm_HandSolder" V 3430 12550 50  0001 C CNN
+F 2 "Resistor_SMD:R_0603_1608Metric_Pad0.98x0.95mm_HandSolder" V 3430 12550 50  0001 C CNN
 F 3 "https://www.yageo.com/upload/media/product/productsearch/datasheet/rchip/PYu-RT_1-to-0.01_RoHS_L_12.pdf" H 3500 12550 50  0001 C CNN
 F 4 "YAG1756CT-ND‎" H 3500 12550 50  0001 C CNN "Digikey"
@@
 F 0 "R6" H -70 10254 50  0000 R CNN
 F 1 "10k" H -70 10345 50  0000 R CNN
-F 2 "Resistor_SMD:R_0201_0603Metric_Pad0.64x0.40mm_HandSolder" V -70 10300 50  0001 C CNN
+F 2 "Resistor_SMD:R_0603_1608Metric_Pad0.98x0.95mm_HandSolder" V -70 10300 50  0001 C CNN
 F 3 "https://www.yageo.com/upload/media/product/productsearch/datasheet/rchip/PYu-RC_Group_51_RoHS_L_11.pdf" H 0   10300 50  0001 C CNN
 F 4 "13-RC0603DR-0710KLCT-ND‎" V 0   10300 50  0001 C CNN "Digikey"
@@
 F 0 "R17" V 3243 9850 50  0000 C CNN
 F 1 "10k" V 3334 9850 50  0000 C CNN
-F 2 "Resistor_SMD:R_0201_0603Metric_Pad0.64x0.40mm_HandSolder" V 3380 9850 50  0001 C CNN
+F 2 "Resistor_SMD:R_0603_1608Metric_Pad0.98x0.95mm_HandSolder" V 3380 9850 50  0001 C CNN
 F 3 "https://www.yageo.com/upload/media/product/productsearch/datasheet/rchip/PYu-RC_Group_51_RoHS_L_11.pdf" H 3450 9850 50  0001 C CNN
 F 4 "13-RC0603DR-0710KLCT-ND‎" V 3450 9850 50  0001 C CNN "Digikey"
@@
 F 0 "R13" H 2730 13554 50  0000 R CNN
 F 1 "10k" H 2730 13645 50  0000 R CNN
-F 2 "Resistor_SMD:R_0201_0603Metric_Pad0.64x0.40mm_HandSolder" V 2730 13600 50  0001 C CNN
+F 2 "Resistor_SMD:R_0603_1608Metric_Pad0.98x0.95mm_HandSolder" V 2730 13600 50  0001 C CNN
 F 3 "https://www.yageo.com/upload/media/product/productsearch/datasheet/rchip/PYu-RC_Group_51_RoHS_L_11.pdf" H 2800 13600 50  0001 C CNN
 F 4 "13-RC0603DR-0710KLCT-ND‎" V 2800 13600 50  0001 C CNN "Digikey"
@@
 F 0 "R19" V 3293 13300 50  0000 C CNN
 F 1 "20k" V 3384 13300 50  0000 C CNN
-F 2 "Resistor_SMD:R_0201_0603Metric_Pad0.64x0.40mm_HandSolder" V 3430 13300 50  0001 C CNN
+F 2 "Resistor_SMD:R_0603_1608Metric_Pad0.98x0.95mm_HandSolder" V 3430 13300 50  0001 C CNN
 F 3 "https://industrial.panasonic.com/cdbs/www-data/pdf/RDM0000/AOA0000C328.pdf" H 3500 13300 50  0001 C CNN
 F 4 "‎P20429CT-ND‎" V 3500 13300 50  0001 C CNN "Digikey"
@@
 F 0 "R8" V 1243 8550 50  0000 C CNN
 F 1 "10k" V 1334 8550 50  0000 C CNN
-F 2 "Resistor_SMD:R_0201_0603Metric_Pad0.64x0.40mm_HandSolder" V 1380 8550 50  0001 C CNN
+F 2 "Resistor_SMD:R_0603_1608Metric_Pad0.98x0.95mm_HandSolder" V 1380 8550 50  0001 C CNN
 F 3 "https://www.yageo.com/upload/media/product/productsearch/datasheet/rchip/PYu-RC_Group_51_RoHS_L_11.pdf" H 1450 8550 50  0001 C CNN
 F 4 "13-RC0603DR-0710KLCT-ND‎" V 1450 8550 50  0001 C CNN "Digikey"
@@
 F 0 "R10" V 1993 9450 50  0000 C CNN
 F 1 "20k" V 2084 9450 50  0000 C CNN
-F 2 "Resistor_SMD:R_0201_0603Metric_Pad0.64x0.40mm_HandSolder" V 2130 9450 50  0001 C CNN
+F 2 "Resistor_SMD:R_0603_1608Metric_Pad0.98x0.95mm_HandSolder" V 2130 9450 50  0001 C CNN
 F 3 "https://industrial.panasonic.com/cdbs/www-data/pdf/RDM0000/AOA0000C328.pdf" H 2200 9450 50  0001 C CNN
 F 4 "‎P20429CT-ND‎" V 2200 9450 50  0001 C CNN "Digikey"
