File: hardware/mallard.sch (KiCad schematic (older format))
At the start: 84 parts, among them J1 USB_A, J2 Conn_02x03_Odd_Even, J3 Conn_01x03, J4 Conn_01x03, J5 Conn_01x03, J6 Conn_01x03, SW1 RESET Switch, U1 TMP235, U10 LTC1983ES6-3, U11 STM32L4Q5xx, U12 LTC3529EDCB, U2 TMP235, U3 TMP235, U4 BQ24210DQCT, U5 TMUX1309, U6 TMUX1309, U7 LMP7721, U8 TPS71710DRVR, U9 LMV554

Commit message: Revised layout, fixed schematic errors
Connections:
- net labels removed: Ref_Elec
- wire segments 287 -> 289
Changed lines of the file:
@@
 Wire Wire Line
 	15450 6250 15500 6250
+Text GLabel 17750 6050 2    50   Input ~ 0
+Eh_Sense
 Text GLabel 17750 5850 2    50   Input ~ 0
-Eh_Sense
+Temp_Sense
 Text GLabel 17750 5950 2    50   Input ~ 0
-Temp_Sense
-Text GLabel 17750 6050 2    50   Input ~ 0
-Ref_Elec
-Text GLabel 17750 6150 2    50   Input ~ 0
-Moisture_Sense
+Ref_Out
 Text Label 17750 6950 0    50   ~ 0
 USB+
@@
 Wire Wire Line
 	17750 7250 17650 7250
-Text GLabel 17750 6250 2    50   Input ~ 0
+Text GLabel 16350 5850 0    50   Input ~ 0
 MUX1_EN
-Text GLabel 17750 6350 2    50   Input ~ 0
+Text GLabel 17750 6550 2    50   Input ~ 0
 MUX1_A0
 Text GLabel 17750 6450 2    50   Input ~ 0
 MUX1_A1
-Text GLabel 16350 5850 0    50   Input ~ 0
+Text GLabel 17750 6350 2    50   Input ~ 0
 MUX2_EN
 Wire Wire Line
-	17750 5850 17650 5850
-Wire Wire Line
-	17650 5950 17750 5950
-Wire Wire Line
 	17750 6050 17650 6050
 Wire Wire Line
-	17650 6150 17750 6150
-Wire Wire Line
-	17750 6250 17650 6250
-Wire Wire Line
-	17650 6350 17750 6350
+	17650 5850 17750 5850
+Wire Wire Line
+	17750 5950 17650 5950
+Wire Wire Line
+	16350 5850 16450 5850
+Wire Wire Line
+	17650 6550 17750 6550
 Wire Wire Line
 	17750 6450 17650 6450
-Text GLabel 16350 5950 0    50   Input ~ 0
+Text GLabel 17750 6250 2    50   Input ~ 0
 MUX2_A0
-Text GLabel 16350 6050 0    50   Input ~ 0
+Text GLabel 17750 6150 2    50   Input ~ 0
 MUX2_A1
 Wire Wire Line
-	16350 5850 16450 5850
-Wire Wire Line
-	16450 5950 16350 5950
-Wire Wire Line
-	16350 6050 16450 6050
+	17750 6350 17650 6350
+Wire Wire Line
+	17650 6250 17750 6250
+Wire Wire Line
+	17750 6150 17650 6150
 Wire Wire Line
 	16000 6250 16450 6250
@@
 L power:GND #PWR0172
 U 1 1 62158AAE
-P 3600 6500
-F 0 "#PWR0172" H 3600 6250 50  0001 C CNN
-F 1 "GND" H 3605 6327 50  0000 C CNN
-F 2 "" H 3600 6500 50  0001 C CNN
-F 3 "" H 3600 6500 50  0001 C CNN
-	1    3600 6500
-	1    0    0    -1
-$EndComp
-Connection ~ 3600 6500
+P 3600 6650
+F 0 "#PWR0172" H 3600 6400 50  0001 C CNN
+F 1 "GND" H 3605 6477 50  0000 C CNN
+F 2 "" H 3600 6650 50  0001 C CNN
+F 3 "" H 3600 6650 50  0001 C CNN
+	1    3600 6650
+	1    0    0    -1
+$EndComp
 Connection ~ 3600 6300
 $Comp
@@
 	1    0    0    -1
 $EndComp
+Wire Wire Line
+	16450 5950 16350 5950
+Text GLabel 16350 5950 0    50   Input ~ 0
+Moisture_Sense
+Wire Wire Line
+	3600 6500 3600 6650
+Connection ~ 3600 6500
+Wire Wire Line
+	3200 6650 3600 6650
+Connection ~ 3600 6650
 $EndSCHEMATC

Commit message: Changes some components on BOM
Parts:
- D1: Digikey S1B-13-F -> S1B-FDICT-ND
- R10, R16, R19: Digikey ‎P20429CT-ND‎ -> P20429CT-ND
- R13, R17, R24, R4, R6, R8: Digikey 13-RC0603DR-0710KLCT-ND‎ -> 13-RC0603DR-0710KLCT-ND
- R15: Digikey 311-30KDCT-ND‎ -> 311-30KDCT-ND
- R18: Digikey YAG1756CT-ND‎ -> YAG1756CT-ND
- U1, U2, U3: symbol mallard:TMP235 -> mallard-rescue:TMP235-mallard
- U10: symbol mallard:LTC1983ES6-3 -> mallard-rescue:LTC1983ES6-3-mallard
- U12: symbol mallard:LTC3529EDCB -> mallard-rescue:LTC3529EDCB-mallard; Digikey LTC3529EDCB#TRPBF -> 161-LTC3529EDCB#TRPBFCT-ND
- U4: symbol mallard:BQ24210DQCT -> mallard-rescue:BQ24210DQCT-mallard
- U5, U6: symbol mallard:TMUX1309 -> mallard-rescue:TMUX1309-mallard; Digikey 296-TMUX1309BQBRCT-ND‎ -> 296-TMUX1309BQBRCT-ND
- U7: symbol mallard:LMP7721 -> mallard-rescue:LMP7721-mallard
- U8: symbol mallard:TPS717 -> mallard-rescue:TPS717-mallard
- U9: symbol mallard:LMV554 -> mallard-rescue:LMV554-mallard
Changed lines of the file:
@@
 F 2 "Resistor_SMD:R_0603_1608Metric_Pad0.98x0.95mm_HandSolder" H 17450 2300 50  0001 C CNN
 F 3 "https://www.yageo.com/upload/media/product/productsearch/datasheet/rchip/PYu-RC_Group_51_RoHS_L_11.pdf" H 17450 2300 50  0001 C CNN
-F 4 "13-RC0603DR-0710KLCT-ND‎" V 17450 2300 50  0001 C CNN "Digikey"
+F 4 "13-RC0603DR-0710KLCT-ND" V 17450 2300 50  0001 C CNN "Digikey"
 	1    17450 2300
 	-1   0    0    1
@@
 	2850 10850 3100 10850
 $Comp
-L mallard:TMUX1309 U?
+L mallard-rescue:TMUX1309-mallard U?
 U 1 1 61FEB939
 P -1350 9250
@@
 F 2 "Package_DFN_QFN:WQFN-16-1EP_3x3mm_P0.5mm_EP1.6x1.6mm" H -1350 7350 50  0001 C CNN
 F 3 "https://www.ti.com/lit/ds/symlink/tmux1309.pdf" H -1350 9250 50  0001 C CNN
-F 4 "296-TMUX1309BQBRCT-ND‎" H -1350 9250 50  0001 C CNN "Digikey"
+F 4 "296-TMUX1309BQBRCT-ND" H -1350 9250 50  0001 C CNN "Digikey"
 	1    -1350 9250
 	1    0    0    -1
@@
 F 2 "Resistor_SMD:R_0603_1608Metric_Pad0.98x0.95mm_HandSolder" V -720 10550 50  0001 C CNN
 F 3 "https://www.yageo.com/upload/media/product/productsearch/datasheet/rchip/PYu-RC_Group_51_RoHS_L_11.pdf" H -650 10550 50  0001 C CNN
-F 4 "13-RC0603DR-0710KLCT-ND‎" V -650 10550 50  0001 C CNN "Digikey"
+F 4 "13-RC0603DR-0710KLCT-ND" V -650 10550 50  0001 C CNN "Digikey"
 	1    -650 10550
 	0    1    1    0
@@
 F 2 "Resistor_SMD:R_0603_1608Metric_Pad0.98x0.95mm_HandSolder" V 3380 9450 50  0001 C CNN
 F 3 "https://industrial.panasonic.com/cdbs/www-data/pdf/RDM0000/AOA0000C328.pdf" H 3450 9450 50  0001 C CNN
-F 4 "‎P20429CT-ND‎" V 3450 9450 50  0001 C CNN "Digikey"
+F 4 "P20429CT-ND" V 3450 9450 50  0001 C CNN "Digikey"
 	1    3450 9450
 	0    1    1    0
@@
 F 2 "Resistor_SMD:R_0603_1608Metric_Pad0.98x0.95mm_HandSolder" V 3380 9050 50  0001 C CNN
 F 3 "https://www.yageo.com/upload/media/product/productsearch/datasheet/rchip/PYu-RT_1-to-0.01_RoHS_L_12.pdf" H 3450 9050 50  0001 C CNN
-F 4 "311-30KDCT-ND‎" V 3450 9050 50  0001 C CNN "Digikey"
+F 4 "311-30KDCT-ND" V 3450 9050 50  0001 C CNN "Digikey"
 	1    3450 9050
 	0    1    1    0
 $EndComp
 $Comp
-L mallard:LMV554 U?
+L mallard-rescue:LMV554-mallard U?
 U 1 1 61FEB955
 P 3500 10200
@@
 F 2 "Resistor_SMD:R_0603_1608Metric_Pad0.98x0.95mm_HandSolder" V 3430 12550 50  0001 C CNN
 F 3 "https://www.yageo.com/upload/media/product/productsearch/datasheet/rchip/PYu-RT_1-to-0.01_RoHS_L_12.pdf" H 3500 12550 50  0001 C CNN
-F 4 "YAG1756CT-ND‎" H 3500 12550 50  0001 C CNN "Digikey"
+F 4 "YAG1756CT-ND" H 3500 12550 50  0001 C CNN "Digikey"
 	1    3500 12550
 	0    1    1    0
@@
 F 2 "Resistor_SMD:R_0603_1608Metric_Pad0.98x0.95mm_HandSolder" V -70 10300 50  0001 C CNN
 F 3 "https://www.yageo.com/upload/media/product/productsearch/datasheet/rchip/PYu-RC_Group_51_RoHS_L_11.pdf" H 0   10300 50  0001 C CNN
-F 4 "13-RC0603DR-0710KLCT-ND‎" V 0   10300 50  0001 C CNN "Digikey"
+F 4 "13-RC0603DR-0710KLCT-ND" V 0   10300 50  0001 C CNN "Digikey"
 	1    0    10300
 	-1   0    0    1
@@
 F 2 "Resistor_SMD:R_0603_1608Metric_Pad0.98x0.95mm_HandSolder" V 3380 9850 50  0001 C CNN
 F 3 "https://www.yageo.com/upload/media/product/productsearch/datasheet/rchip/PYu-RC_Group_51_RoHS_L_11.pdf" H 3450 9850 50  0001 C CNN
-F 4 "13-RC0603DR-0710KLCT-ND‎" V 3450 9850 50  0001 C CNN "Digikey"
+F 4 "13-RC0603DR-0710KLCT-ND" V 3450 9850 50  0001 C CNN "Digikey"
 	1    3450 9850
 	0    1    1    0
@@
 F 2 "Resistor_SMD:R_0603_1608Metric_Pad0.98x0.95mm_HandSolder" V 2730 13600 50  0001 C CNN
 F 3 "https://www.yageo.com/upload/media/product/productsearch/datasheet/rchip/PYu-RC_Group_51_RoHS_L_11.pdf" H 2800 13600 50  0001 C CNN
-F 4 "13-RC0603DR-0710KLCT-ND‎" V 2800 13600 50  0001 C CNN "Digikey"
+F 4 "13-RC0603DR-0710KLCT-ND" V 2800 13600 50  0001 C CNN "Digikey"
 	1    2800 13600
 	-1   0    0    1
@@
 F 2 "Resistor_SMD:R_0603_1608Metric_Pad0.98x0.95mm_HandSolder" V 3430 13300 50  0001 C CNN
 F 3 "https://industrial.panasonic.com/cdbs/www-data/pdf/RDM0000/AOA0000C328.pdf" H 3500 13300 50  0001 C CNN
-F 4 "‎P20429CT-ND‎" V 3500 13300 50  0001 C CNN "Digikey"
+F 4 "P20429CT-ND" V 3500 13300 50  0001 C CNN "Digikey"
 	1    3500 13300
 	0    1    1    0
@@
 Ref_Out
 $Comp
-L mallard:TMUX1309 U?
+L mallard-rescue:TMUX1309-mallard U?
 U 1 1 61FEB9A9
 P -1300 11650
@@
 F 2 "Package_DFN_QFN:WQFN-16-1EP_3x3mm_P0.5mm_EP1.6x1.6mm" H -1300 9750 50  0001 C CNN
 F 3 "https://www.ti.com/lit/ds/symlink/tmux1309.pdf" H -1300 11650 50  0001 C CNN
-F 4 "296-TMUX1309BQBRCT-ND‎" H -1300 11650 50  0001 C CNN "Digikey"
+F 4 "296-TMUX1309BQBRCT-ND" H -1300 11650 50  0001 C CNN "Digikey"
 	1    -1300 11650
 	1    0    0    -1
@@
 	-1700 12250 -1800 12250
 $Comp
-L mallard:TMP235 U?
+L mallard-rescue:TMP235-mallard U?
 U 1 1 61FEB9BC
 P -5100 12450
@@
 $EndComp
 $Comp
-L mallard:TMP235 U?
+L mallard-rescue:TMP235-mallard U?
 U 1 1 61FEB9DC
 P -5100 13350
@@
 $EndComp
 $Comp
-L mallard:TMP235 U?
+L mallard-rescue:TMP235-mallard U?
 U 1 1 61FEB9FC
 P -5150 14200
@@
 F 2 "Resistor_SMD:R_0603_1608Metric_Pad0.98x0.95mm_HandSolder" V 2130 9450 50  0001 C CNN
 F 3 "https://industrial.panasonic.com/cdbs/www-data/pdf/RDM0000/AOA0000C328.pdf" H 2200 9450 50  0001 C CNN
-F 4 "‎P20429CT-ND‎" V 2200 9450 50  0001 C CNN "Digikey"
+F 4 "P20429CT-ND" V 2200 9450 50  0001 C CNN "Digikey"
 	1    2200 9450
 	0    1    1    0
@@
 $EndComp
 $Comp
-L mallard:BQ24210DQCT U4
+L mallard-rescue:BQ24210DQCT-mallard U4
 U 1 1 620370F3
 P 3550 2900
@@
 $EndComp
 $Comp
-L mallard:LTC1983ES6-3 U10
+L mallard-rescue:LTC1983ES6-3-mallard U10
 U 1 1 620370FA
 P 9300 2900
@@
 F 2 "Diode_SMD:D_SMA_Handsoldering" H 1600 3000 50  0001 C CNN
 F 3 "https://www.diodes.com/assets/Datasheets/ds16003.pdf" H 1600 3000 50  0001 C CNN
-F 4 "S1B-13-F" H 1600 3000 50  0001 C CNN "Digikey"
+F 4 "S1B-FDICT-ND" H 1600 3000 50  0001 C CNN "Digikey"
 	1    1600 3000
 	-1   0    0    1
@@
 +1V0_EN
 $Comp
-L mallard:TPS717 U8
+L mallard-rescue:TPS717-mallard U8
 U 1 1 6203711F
 P 9100 4350
@@
 Wrong footprint size
 $Comp
-L mallard:LTC3529EDCB U12
+L mallard-rescue:LTC3529EDCB-mallard U12
 U 1 1 62066D6A
 P 2400 5950
@@
 F 2 "mallard:DFN200X300X80-9N" H 2300 6100 50  0001 C CNN
 F 3 "https://www.analog.com/media/en/technical-documentation/data-sheets/3529fb.pdf" H 2300 6100 50  0001 C CNN
-F 4 "LTC3529EDCB#TRPBF" H 2400 5950 50  0001 C CNN "Digikey"
+F 4 "161-LTC3529EDCB#TRPBFCT-ND" H 2400 5950 50  0001 C CNN "Digikey"
 	1    2400 5950
 	1    0    0    -1
@@
 F 2 "Resistor_SMD:R_0603_1608Metric_Pad0.98x0.95mm_HandSolder" V 1380 8550 50  0001 C CNN
 F 3 "https://www.yageo.com/upload/media/product/productsearch/datasheet/rchip/PYu-RC_Group_51_RoHS_L_11.pdf" H 1450 8550 50  0001 C CNN
-F 4 "13-RC0603DR-0710KLCT-ND‎" V 1450 8550 50  0001 C CNN "Digikey"
+F 4 "13-RC0603DR-0710KLCT-ND" V 1450 8550 50  0001 C CNN "Digikey"
 	1    1450 8550
 	0    1    1    0
@@
 $EndComp
 $Comp
-L mallard:LMP7721 U?
+L mallard-rescue:LMP7721-mallard U?
 U 1 1 61FEBA54
 P 1450 9450
